Commit message: chore: clean up redundant packages and duplicate files
- Delete deprecated packages: hand_eye_calibration, jaka_hardware,
  swap_fsm, visual_servo (not relevant for ZU7 thesis project)
- Delete duplicate world files from root and src directories
- Delete obsolete launch files and models
- Update progress.md

Co-Authored-By: Claude Opus 4.6 <noreply@anthropic.com>

File: src/jaka_vision/urdf/inc/jaka_camera_gazebo.xacro (robot description, xacro)
@@ -1,17 +1,51 @@
 <?xml version="1.0"?>
 <!--
-  JAKA ZU7 Eye-in-Hand Camera Configuration for Gazebo Sim (Fortress)
+  JAKA ZU7 Camera Configuration for Gazebo Sim (Fortress)
+  Support for multiple camera types and mounting positions
   Usage in robot URDF xacro:
     <xacro:include filename="$(find jaka_vision)/urdf/inc/jaka_camera_gazebo.xacro" />
-    <xacro:jaka_camera_gazebo parent="Link_6" />
+    OR with custom parameters:
+    <xacro:jaka_camera_gazebo
+        parent="Link_6"
+        camera_type="realsense"
+        offset_x="0.0" offset_y="0.0" offset_z="0.05"
+        offset_roll="0.0" offset_pitch="0.0" offset_yaw="0.0" />
+  Parameters:
+    parent          - Parent link to attach camera (default: Link_6)
+    camera_type     - Camera model: realsense_d435 / kinect / generic (default: generic)
+    offset_x/y/z    - Position offset from parent link (default: 0.0 0.0 0.05)
+    offset_roll/pitch/yaw - Rotation offset in radians (default: 0 0 0)
+    joint_type      - Joint type: fixed / floating / revolute (default: fixed)
+    camera_name     - Camera namespace (default: camera)
+    update_rate     - Camera update rate Hz (default: 30.0)
+    image_width     - Image width pixels (default: 640)
+    image_height    - Image height pixels (default: 480)
+    update_rate     - Sensor update rate (default: 30.0)
 -->
 <robot xmlns:xacro="http://wiki.ros.org/xacro"
        xmlns:gazebo="http://gazebosim.org">
-    <xacro:macro name="jaka_camera_gazebo" params="parent">
-        <!-- Camera optical frame link -->
-        <link name="camera_link_optical">
+    <!-- Camera type definitions -->
+    <xacro:property name="REALSENSE_D435" value="realsense_d435" />
+    <xacro:property name="KINECT" value="kinect" />
+    <xacro:property name="GENERIC" value="generic" />
+    <xacro:macro name="jaka_camera_gazebo" params="parent:=Link_6
+                                                  camera_type:=generic
+                                                  offset_x:=0.0 offset_y:=0.0 offset_z:=0.05
+                                                  offset_roll:=0.0 offset_pitch:=0.0 offset_yaw:=0.0
+                                                  joint_type:=fixed
+                                                  camera_name:=camera
+                                                  update_rate:=30.0
+                                                  image_width:=640
+                                                  image_height:=480">
+        <!-- Calculate camera visual dimensions based on type -->
+        <xacro:property name="camera_box_size"
+                       value="${'0.025 0.09 0.025' if camera_type == REALSENSE_D435 else ('0.06 0.18 0.07' if camera_type == KINECT else '0.02 0.02 0.02')}" />
+        <xacro:property name="camera_box_color"
+                       value="${'0.3 0.3 0.3 1.0' if camera_type == REALSENSE_D435 else ('0.2 0.4 0.6 1.0' if camera_type == KINECT else '0.1 0.1 0.1 1.0')}" />
+        <!-- Camera optical frame link (ROS convention: -90deg roll) -->
+        <link name="${camera_name}_link_optical">
         </link>
         <!-- Camera physical link -->
-        <link name="camera_link">
+        <link name="${camera_name}_link">
             <inertial>
                 <origin xyz="0 0 0" rpy="0 0 0" />
@@ -22,8 +56,8 @@
                 <origin xyz="0 0 0" rpy="0 0 0" />
                 <geometry>
-                    <box size="0.02 0.02 0.02" />
+                    <box size="${camera_box_size}" />
                 </geometry>
-                <material name="black">
-                    <color rgba="0.1 0.1 0.1 1.0" />
+                <material name="${camera_name}_black">
+                    <color rgba="${camera_box_color}" />
                 </material>
             </visual>
@@ -31,41 +65,86 @@
                 <origin xyz="0 0 0" rpy="0 0 0" />
                 <geometry>
-                    <box size="0.02 0.02 0.02" />
+                    <box size="${camera_box_size}" />
                 </geometry>
             </collision>
         </link>
-        <!-- Fixed joint to parent (end-effector) -->
-        <joint name="camera_joint" type="fixed">
-            <origin xyz="0.0 0.0 0.05" rpy="0 0 0" />
+        <!-- Joint to parent (end-effector) - configurable type -->
+        <joint name="${camera_name}_joint" type="${joint_type}">
+            <origin xyz="${offset_x} ${offset_y} ${offset_z}" rpy="${offset_roll} ${offset_pitch} ${offset_yaw}" />
             <parent link="${parent}" />
-            <child link="camera_link" />
+            <child link="${camera_name}_link" />
+            <!-- Only add dynamics for non-fixed joints -->
+            <xacro:if value="${joint_type != 'fixed'}">
+                <dynamics damping="0.1" friction="0.1" />
+            </xacro:if>
         </joint>
-        <!-- Optical frame joint for ROS convention -->
-        <joint name="camera_optical_joint" type="fixed">
+        <!-- Optical frame joint for ROS convention (ROS uses: X=forward, Y=left, Z=up) -->
+        <!-- Gazebo camera: X=right, Y=down, Z=forward -->
+        <!-- Transform: Roll=-90deg, Pitch=0, Yaw=-90deg -->
+        <joint name="${camera_name}_optical_joint" type="fixed">
             <origin xyz="0.0 0.0 0.0" rpy="-1.5707 0 -1.5707"/>
-            <parent link="camera_link"/>
-            <child link="camera_link_optical"/>
+            <parent link="${camera_name}_link"/>
+            <child link="${camera_name}_link_optical"/>
         </joint>
         <!-- Gazebo sensor configuration -->
-        <gazebo reference="camera_link">
-            <sensor name="camera_sensor" type="camera">
+        <gazebo reference="${camera_name}_link">
+            <sensor name="${camera_name}_sensor" type="camera">
                 <always_on>true</always_on>
-                <update_rate>30.0</update_rate>
+                <update_rate>${update_rate}</update_rate>
                 <visualize>true</visualize>
                 <camera>
-                    <horizontal_fov>1.047</horizontal_fov>
+                    <!-- FOV based on camera type -->
+                    <horizontal_fov>${'1.396' if camera_type == REALSENSE_D435 else ('1.047' if camera_type == KINECT else '1.047')}</horizontal_fov>
                     <image>
-                        <width>640</width>
-                        <height>480</height>
+                        <width>${image_width}</width>
+                        <height>${image_height}</height>
                         <format>R8G8B8</format>
                     </image>
                     <clip>
-                        <near>0.05</near>
-                        <far>10.0</far>
+                        <near>${'0.1' if camera_type == REALSENSE_D435 else ('0.5' if camera_type == KINECT else '0.05')}</near>
+                        <far>${'10.0' if camera_type == REALSENSE_D435 else ('10.0' if camera_type == KINECT else '10.0')}</far>
                     </clip>
+                    <!-- Distortion for Kinect -->
+                    <xacro:if value="${camera_type == KINECT}">
+                        <distortion>
+                            <k1>0.0</k1>
+                            <k2>0.0</k2>
+                            <k3>0.0</k3>
+                            <p1>0.0</p1>
+                            <p2>0.0</p2>
+                            <cx>0.0</cx>
+                            <cy>0.0</cy>
+                        </distortion>
+                    </xacro:if>
                 </camera>
-                <topic>/camera/image_raw</topic>
+                <topic>${camera_name}/image_raw</topic>
             </sensor>
         </gazebo>
     </xacro:macro>
+    <!-- Convenience macro: Realsense D435 (common eye-in-hand camera) -->
+    <xacro:macro name="jaka_camera_realsense" params="parent:=Link_6 offset_x:=0.0 offset_y:=0.0 offset_z:=0.02">
+        <xacro:jaka_camera_gazebo
+            parent="${parent}"
+            camera_type="realsense_d435"
+            offset_x="${offset_x}" offset_y="${offset_y}" offset_z="${offset_z}"
+            offset_roll="0.0" offset_pitch="0.0" offset_yaw="0.0"
+            joint_type="fixed"
+            camera_name="camera"
+            update_rate="30.0"
+            image_width="640"
+            image_height="480" />
+    </xacro:macro>
+    <!-- Convenience macro: Kinect (external/mounted camera) -->
+    <xacro:macro name="jaka_camera_kinect" params="parent:=world offset_x:=0.5 offset_y:=0.0 offset_z:=1.0">
+        <xacro:jaka_camera_gazebo
+            parent="${parent}"
+            camera_type="kinect"
+            offset_x="${offset_x}" offset_y="${offset_y}" offset_z="${offset_z}"
+            offset_roll="0.0" offset_pitch="0.0" offset_yaw="0.0"
+            joint_type="fixed"
+            camera_name="camera"
+            update_rate="30.0"
+            image_width="640"
+            image_height="480" />
+    </xacro:macro>
 </robot>

File: src/jaka_zu7_moveit_config/config/jaka_zu7_with_camera.urdf.xacro (robot description, xacro)
@@ -1,15 +1,62 @@
 <?xml version="1.0"?>
+<!--
+  JAKA ZU7 with Configurable Camera
+  Parameters:
+    initial_positions_file  - YAML file with initial joint positions
+    use_gazebo             - Use Gazebo simulation (default: false)
+    use_rviz_sim           - Use RViz simulation mode (default: false)
+  Camera Parameters (for eye-in-hand):
+    camera_type            - Camera model: realsense_d435 / kinect / generic (default: generic)
+    camera_offset_x/y/z    - Camera position offset from Link_6 (default: 0.0 0.0 0.05)
+    camera_offset_roll/pitch/yaw - Camera rotation offset (default: 0 0 0)
+    camera_joint_type      - Joint type: fixed / floating / revolute (default: fixed)
+    camera_update_rate     - Camera update rate Hz (default: 30.0)
+    camera_image_width/height - Image resolution (default: 640 480)
+  Usage Examples:
+    1. Default generic camera at 5cm above Link_6:
+       <xacro:include filename="jaka_zu7_with_camera.urdf.xacro" />
+    2. Realsense D435 at custom offset:
+       ros2 launch ... robot_description:=$(find jaka_zu7_moveit_config)/config/jaka_zu7_with_camera.urdf.xacro
+       camera_type:=realsense_d435 camera_offset_z:=0.02
+    3. Floating camera (simulate hand-eye freedom):
+       camera_joint_type:=floating
+-->
 <robot xmlns:xacro="http://www.ros.org/wiki/xacro" name="jaka_zu7">
+    <!-- Standard robot arguments -->
     <xacro:arg name="initial_positions_file" default="initial_positions.yaml" />
     <xacro:arg name="use_gazebo" default="false"/>
     <xacro:arg name="use_rviz_sim" default="false"/>
+    <!-- Camera configuration arguments -->
+    <xacro:arg name="camera_type" default="generic"/>
+    <xacro:arg name="camera_offset_x" default="0.0"/>
+    <xacro:arg name="camera_offset_y" default="0.0"/>
+    <xacro:arg name="camera_offset_z" default="0.05"/>
+    <xacro:arg name="camera_offset_roll" default="0.0"/>
+    <xacro:arg name="camera_offset_pitch" default="0.0"/>
+    <xacro:arg name="camera_offset_yaw" default="0.0"/>
+    <xacro:arg name="camera_joint_type" default="fixed"/>
+    <xacro:arg name="camera_update_rate" default="30.0"/>
+    <xacro:arg name="camera_image_width" default="640"/>
+    <xacro:arg name="camera_image_height" default="480"/>
     <!-- Import jaka_zu7 urdf file -->
     <xacro:include filename="$(find jaka_description)/urdf/jaka_zu7.urdf" />
     <!-- Import control_xacro -->
     <xacro:include filename="jaka_zu7.ros2_control.xacro" />
-    <!-- Import camera xacro (eye-in-hand) -->
+    <!-- Import camera xacro -->
     <xacro:include filename="$(find jaka_vision)/urdf/inc/jaka_camera_gazebo.xacro" />
-    <!-- Add camera to end-effector (tool0 = Link_6) -->
-    <xacro:jaka_camera_gazebo parent="Link_6" />
+    <!-- Add camera to end-effector (Link_6) with configurable parameters -->
+    <xacro:jaka_camera_gazebo
+        parent="Link_6"
+        camera_type="$(arg camera_type)"
+        offset_x="$(arg camera_offset_x)"
+        offset_y="$(arg camera_offset_y)"
+        offset_z="$(arg camera_offset_z)"
+        offset_roll="$(arg camera_offset_roll)"
+        offset_pitch="$(arg camera_offset_pitch)"
+        offset_yaw="$(arg camera_offset_yaw)"
+        joint_type="$(arg camera_joint_type)"
+        update_rate="$(arg camera_update_rate)"
+        image_width="$(arg camera_image_width)"
+        image_height="$(arg camera_image_height)" />
     <!-- ros2_control hardware -->
     <xacro:jaka_zu7_ros2_control name="jaka_zu7_hardware" initial_positions_file="$(arg initial_positions_file)" use_gazebo="$(arg use_gazebo)" use_rviz_sim="$(arg use_rviz_sim)" />
